File: Teebeutel-Expansion-Blank.kicad_pcb (KiCad board)
At the start: 2 copper layers, 72 x 100 mm, 6 parts, among them J1 Conn_01x10_Male, J2 Conn_01x10_Female, J3 Conn_01x10_Male, J4 Conn_01x10_Female

Commit message: chore: cleanup and update to KiCad6
Other:
- net class Default removed

Commit message: chore: Update labels
Connections:
- J3 pad 2: IO0 -> IO7
- J3 pad 3: IO1 -> IO6
- J3 pad 4: IO2 -> IO5
- J3 pad 5: IO3 -> IO4
- J3 pad 6: IO4 -> IO3
- J3 pad 7: IO5 -> IO2
- J3 pad 8: IO6 -> IO1
- J3 pad 9: IO7 -> IO0
- J4 pad 2: IO0 -> IO7
- J4 pad 3: IO1 -> IO6
- J4 pad 4: IO2 -> IO5
- J4 pad 5: IO3 -> IO4
- J4 pad 6: IO4 -> IO3
- J4 pad 7: IO5 -> IO2
- J4 pad 8: IO6 -> IO1
- J4 pad 9: IO7 -> IO0
Changed lines of the file:
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@@
       (net 10 "+3V3"))
     (pad "2" thru_hole oval locked (at 0 2.54) (size 1.7 1.7) (drill 1) (layers *.Cu *.Mask)
+      (net 11 "IO7"))
+    (pad "3" thru_hole oval locked (at 0 5.08) (size 1.7 1.7) (drill 1) (layers *.Cu *.Mask)
+      (net 12 "IO6"))
+    (pad "4" thru_hole oval locked (at 0 7.62) (size 1.7 1.7) (drill 1) (layers *.Cu *.Mask)
+      (net 13 "IO5"))
+    (pad "5" thru_hole oval locked (at 0 10.16) (size 1.7 1.7) (drill 1) (layers *.Cu *.Mask)
+      (net 14 "IO4"))
+    (pad "6" thru_hole oval locked (at 0 12.7) (size 1.7 1.7) (drill 1) (layers *.Cu *.Mask)
+      (net 15 "IO3"))
+    (pad "7" thru_hole oval locked (at 0 15.24) (size 1.7 1.7) (drill 1) (layers *.Cu *.Mask)
+      (net 16 "IO2"))
+    (pad "8" thru_hole oval locked (at 0 17.78) (size 1.7 1.7) (drill 1) (layers *.Cu *.Mask)
+      (net 17 "IO1"))
+    (pad "9" thru_hole oval locked (at 0 20.32) (size 1.7 1.7) (drill 1) (layers *.Cu *.Mask)
       (net 18 "IO0"))
-    (pad "3" thru_hole oval locked (at 0 5.08) (size 1.7 1.7) (drill 1) (layers *.Cu *.Mask)
-      (net 17 "IO1"))
-    (pad "4" thru_hole oval locked (at 0 7.62) (size 1.7 1.7) (drill 1) (layers *.Cu *.Mask)
-      (net 16 "IO2"))
-    (pad "5" thru_hole oval locked (at 0 10.16) (size 1.7 1.7) (drill 1) (layers *.Cu *.Mask)
-      (net 15 "IO3"))
-    (pad "6" thru_hole oval locked (at 0 12.7) (size 1.7 1.7) (drill 1) (layers *.Cu *.Mask)
-      (net 14 "IO4"))
-    (pad "7" thru_hole oval locked (at 0 15.24) (size 1.7 1.7) (drill 1) (layers *.Cu *.Mask)
-      (net 13 "IO5"))
-    (pad "8" thru_hole oval locked (at 0 17.78) (size 1.7 1.7) (drill 1) (layers *.Cu *.Mask)
-      (net 12 "IO6"))
-    (pad "9" thru_hole oval locked (at 0 20.32) (size 1.7 1.7) (drill 1) (layers *.Cu *.Mask)
-      (net 11 "IO7"))
     (pad "10" thru_hole oval locked (at 0 22.86) (size 1.7 1.7) (drill 1) (layers *.Cu *.Mask)
       (net 1 "GND"))
@@
       (net 10 "+3V3"))
     (pad "2" thru_hole oval locked (at 0 -2.54 180) (size 1.7 1.7) (drill 1) (layers *.Cu *.Mask)
+      (net 11 "IO7"))
+    (pad "3" thru_hole oval locked (at 0 -5.08 180) (size 1.7 1.7) (drill 1) (layers *.Cu *.Mask)
+      (net 12 "IO6"))
+    (pad "4" thru_hole oval locked (at 0 -7.62 180) (size 1.7 1.7) (drill 1) (layers *.Cu *.Mask)
+      (net 13 "IO5"))
+    (pad "5" thru_hole oval locked (at 0 -10.16 180) (size 1.7 1.7) (drill 1) (layers *.Cu *.Mask)
+      (net 14 "IO4"))
+    (pad "6" thru_hole oval locked (at 0 -12.7 180) (size 1.7 1.7) (drill 1) (layers *.Cu *.Mask)
+      (net 15 "IO3"))
+    (pad "7" thru_hole oval locked (at 0 -15.24 180) (size 1.7 1.7) (drill 1) (layers *.Cu *.Mask)
+      (net 16 "IO2"))
+    (pad "8" thru_hole oval locked (at 0 -17.78 180) (size 1.7 1.7) (drill 1) (layers *.Cu *.Mask)
+      (net 17 "IO1"))
+    (pad "9" thru_hole oval locked (at 0 -20.32 180) (size 1.7 1.7) (drill 1) (layers *.Cu *.Mask)
       (net 18 "IO0"))
-    (pad "3" thru_hole oval locked (at 0 -5.08 180) (size 1.7 1.7) (drill 1) (layers *.Cu *.Mask)
-      (net 17 "IO1"))
-    (pad "4" thru_hole oval locked (at 0 -7.62 180) (size 1.7 1.7) (drill 1) (layers *.Cu *.Mask)
-      (net 16 "IO2"))
-    (pad "5" thru_hole oval locked (at 0 -10.16 180) (size 1.7 1.7) (drill 1) (layers *.Cu *.Mask)
-      (net 15 "IO3"))
-    (pad "6" thru_hole oval locked (at 0 -12.7 180) (size 1.7 1.7) (drill 1) (layers *.Cu *.Mask)
-      (net 14 "IO4"))
-    (pad "7" thru_hole oval locked (at 0 -15.24 180) (size 1.7 1.7) (drill 1) (layers *.Cu *.Mask)
-      (net 13 "IO5"))
-    (pad "8" thru_hole oval locked (at 0 -17.78 180) (size 1.7 1.7) (drill 1) (layers *.Cu *.Mask)
-      (net 12 "IO6"))
-    (pad "9" thru_hole oval locked (at 0 -20.32 180) (size 1.7 1.7) (drill 1) (layers *.Cu *.Mask)
-      (net 11 "IO7"))
     (pad "10" thru_hole oval locked (at 0 -22.86 180) (size 1.7 1.7) (drill 1) (layers *.Cu *.Mask)
       (net 1 "GND"))
@@
     (effects (font (size 0.7 0.7) (thickness 0.15)))
   )
-  (gr_text "IO7" (at 180.448 100.323 90) (layer "F.SilkS")
-    (effects (font (size 0.7 0.7) (thickness 0.15)))
-  )
-  (gr_text "IO0" (at 180.52 82.543 90) (layer "F.SilkS")
+  (gr_text "IO0" (at 180.448 100.323 90) (layer "F.SilkS")
+    (effects (font (size 0.7 0.7) (thickness 0.15)))
+  )
+  (gr_text "IO7" (at 180.52 82.543 90) (layer "F.SilkS")
     (effects (font (size 0.7 0.7) (thickness 0.15)))
   )
@@
     (effects (font (size 0.7 0.7) (thickness 0.15)))
   )
-  (gr_text "IO5" (at 180.448 95.243 90) (layer "F.SilkS")
-    (effects (font (size 0.7 0.7) (thickness 0.15)))
-  )
-  (gr_text "IO1" (at 180.52 85.083 90) (layer "F.SilkS")
+  (gr_text "IO2" (at 180.448 95.243 90) (layer "F.SilkS")
+    (effects (font (size 0.7 0.7) (thickness 0.15)))
+  )
+  (gr_text "IO6" (at 180.52 85.083 90) (layer "F.SilkS")
     (effects (font (size 0.7 0.7) (thickness 0.15)))
   )
@@
     (effects (font (size 0.7 0.7) (thickness 0.15)))
   )
-  (gr_text "IO6" (at 180.448 97.783 90) (layer "F.SilkS")
+  (gr_text "IO1" (at 180.448 97.783 90) (layer "F.SilkS")
     (effects (font (size 0.7 0.7) (thickness 0.15)))
   )
@@
     (effects (font (size 0.7 0.7) (thickness 0.15)))
   )
-  (gr_text "IO3" (at 180.448 90.163 90) (layer "F.SilkS")
+  (gr_text "IO4" (at 180.448 90.163 90) (layer "F.SilkS")
     (effects (font (size 0.7 0.7) (thickness 0.15)))
   )
@@
     (effects (font (size 0.7 0.7) (thickness 0.15)))
   )
-  (gr_text "IO4" (at 180.448 92.703 90) (layer "F.SilkS")
-    (effects (font (size 0.7 0.7) (thickness 0.15)))
-  )
-  (gr_text "IO2" (at 180.448 87.623 90) (layer "F.SilkS")
-    (effects (font (size 0.7 0.7) (thickness 0.15)))
-  )
+  (gr_text "IO3" (at 180.448 92.703 90) (layer "F.SilkS")
+    (effects (font (size 0.7 0.7) (thickness 0.15)))
+  )
+  (gr_text "IO5" (at 180.448 87.623 90) (layer "F.SilkS")
+    (effects (font (size 0.7 0.7) (thickness 0.15)))
+  )
