File: Teebeutel-Expansion.kicad_pcb (KiCad board)
At the start: 2 copper layers, 72 x 100 mm, 759 parts, among them J1 Conn_01x10_Male, J2 Conn_01x10_Female, J3 Conn_01x10_Male, J4 Conn_01x10_Female, J5 Conn_02x03_Counter_Clockwise, J6 Conn_02x03_Counter_Clockwise, J7 Conn_01x03, J8 Conn_01x03, J9 Conn_02x08_Counter_Clockwise

Commit message: chore: cleanup and update to KiCad6
Other:
- net class Default removed

Commit message: chore: Update labels
Parts:
- TP1, TP10, TP11, TP12, TP13, TP14, TP15, TP16, TP17, TP18, TP19, TP2, TP20, TP21, TP22, TP23, TP24, TP25, TP26, TP27, TP28, TP29, TP3, TP30, TP31, TP32, TP33, TP34, TP35, TP36, TP37, TP38, TP39, TP4, TP40, TP41, TP42, TP43, TP44, TP45, TP46, TP47, TP48, TP49, TP5, TP50, TP6, TP7, TP8, TP9: footprint Teebeutel-Expansion:THTPad_D1.5mm_Drill0.7mm -> TestPoint:TestPoint_THTPad_D1.5mm_Drill0.7mm
Connections:
- J3 pad 2: IO0 -> IO7
- J3 pad 3: IO1 -> IO6
- J3 pad 4: IO2 -> IO5
- J3 pad 5: IO3 -> IO4
- J3 pad 6: IO4 -> IO3
- J3 pad 7: IO5 -> IO2
- J3 pad 8: IO6 -> IO1
- J3 pad 9: IO7 -> IO0
- J4 pad 2: IO0 -> IO7
- J4 pad 3: IO1 -> IO6
- J4 pad 4: IO2 -> IO5
- J4 pad 5: IO3 -> IO4
- J4 pad 6: IO4 -> IO3
- J4 pad 7: IO5 -> IO2
- J4 pad 8: IO6 -> IO1
- J4 pad 9: IO7 -> IO0
- TP10 pad 1: IO1 -> IO6
- TP11 pad 1: IO2 -> IO5
- TP12 pad 1: IO3 -> IO4
- TP13 pad 1: IO4 -> IO3
- TP14 pad 1: IO5 -> IO2
- TP15 pad 1: IO6 -> IO1
- TP16 pad 1: IO7 -> IO0
- TP9 pad 1: IO0 -> IO7
